File: vscp-din-wireless-esp8266.kicad_pcb (KiCad board)
At the start: 2 copper layers, 64.8 x 51 mm, 25 parts, among them J1 Conn_01x04_Left, J2 Conn_01x04_Right, J3 Conn_01x06, J4 Conn_01x02, Q1 BC547, U2 ESP-12E

Commit message: Fixed board to board connector
Parts:
- renumbered R3 to R4
Connections:
- J2 pad 2: Net-(J2-Pad2) -> VCC
- J2 pad 4: VCC -> Net-(J2-Pad4)
Routing:
- net VCC: track 170.2 -> 174.3 mm
