File: vscp-din-wireless-esp8266.sch (KiCad schematic (older format))
At the start: 24 parts, among them J1 Conn_01x04_Left, J2 Conn_01x04_Right, J3 Conn_01x06, J4 Conn_01x02, Q1 BC547, U2 ESP-12E

Commit message: Fixed board to board connector
Connections:
- net VCC: now also J2.2 (Pin_2); no longer J2.4 (Pin_4)
Changed lines of the file:
@@
 $EndComp
-Wire Wire Line
-	4200 6750 4200 6250
 Wire Wire Line
 	8500 5750 6950 5750
@@
 Wire Wire Line
 	3700 6250 4200 6250
-Connection ~ 4200 6250
 Wire Wire Line
 	4200 6250 4200 4700
@@
 Text Label 7400 2750 0    50   ~ 0
 leda
+Wire Wire Line
+	4400 6750 4400 6250
+Wire Wire Line
+	4400 6250 4200 6250
+Connection ~ 4200 6250
 $EndSCHEMATC
